File: loraguide.kicad_pcb (KiCad board)
At the start: 2 copper layers, 30 x 65 mm, 21 parts, among them J1 USB_C_Receptacle_USB2.0_14P, J2 Conn_Coaxial, U1 ESP32-S3-WROOM-1, U2 SX1262IMLTRT, U3 AMS1117-3.3

Commit message: upload
Parts:
- removed BOOT: BOOT, Button_Switch_SMD:SW_SPST_B3U-1000P
- removed RST: RST, Button_Switch_SMD:SW_SPST_B3U-1000P
- added M1: MountingHole_2.7mm_M2.5, MountingHole:MountingHole_2.7mm_M2.5, F.Cu at (154.0, 97.0)
- added M2: MountingHole_2.7mm_M2.5, MountingHole:MountingHole_2.7mm_M2.5, F.Cu at (206.0, 97.0)
- added M3: MountingHole_2.7mm_M2.5, MountingHole:MountingHole_2.7mm_M2.5, F.Cu at (206.0, 66.5)
- added M4: MountingHole_2.7mm_M2.5, MountingHole:MountingHole_2.7mm_M2.5, F.Cu at (154.0, 67.0)
- added SW1: RST, Button_Switch_SMD:SW_SPST_B3U-1000P, F.Cu at (177.2, 98.0)
- added SW2: BOOT, Button_Switch_SMD:SW_SPST_B3U-1000P, F.Cu at (181.5, 98.0)
- added U4: BME280, Package_LGA:Bosch_LGA-8_2.5x2.5mm_P0.65mm_ClockwisePinNumbering, F.Cu at (152.2, 81.5)
- added U5: L80-R, RF_GPS:Quectel_L80-R, F.Cu at (192.5, 72.5)
- L1: footprint Inductor_SMD:L_0402_1005Metric -> Inductor_SMD:L_0603_1608Metric
- moved G1 148.4 mm to (207.0, 81.0), turned to 90 degrees
- moved C3 134.8 mm to (202.0, 88.0), turned to 0 degrees
- moved U2 130.1 mm to (198.2, 84.8), turned to 0 degrees
- moved L1 126.7 mm to (196.0, 90.3), turned to -90 degrees
- moved C5 126.6 mm to (194.5, 82.5), turned to 0 degrees
- moved C2 126.1 mm to (199.5, 92.5), turned to 0 degrees
- moved R3 125.8 mm to (177.0, 94.5), turned to -90 degrees
- moved C1 123.9 mm to (199.5, 90.0), turned to 0 degrees
- moved J2 123.4 mm to (198.5, 96.5)
- moved C4 123.4 mm to (194.5, 88.0), turned to 0 degrees
- moved C7 122.9 mm to (183.5, 88.5)
- moved U3 121.9 mm to (177.0, 89.0)
- moved C6 116.6 mm to (171.5, 92.0), turned to -90 degrees
- moved R2 108.9 mm to (170.5, 97.5)
- moved J1 108.8 mm to (160.7, 94.6)
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Connections:
- U1 pad 18: unconnected-(U1-IO10-Pad18) -> /BME_CS
- U1 pad 36: unconnected-(U1-RXD0-Pad36) -> /TX1
- U1 pad 37: unconnected-(U1-TXD0-Pad37) -> /RX1
Routing:
- net /NSS: track 100.2 -> 71.2 mm, vias 4 -> 2
- net /USB_Data+: track 48.3 -> 21.9 mm
- net /USB_Data-: track 48.2 -> 22.2 mm
- net /MOSI: track 52.9 -> 78.3 mm, vias 2 -> 3
- net /SCK: track 102.5 -> 80.4 mm
- net Net-(J2-In): track 9.35 -> 28.8 mm
- net /MISO: track 102.6 -> 83.2 mm
- net /BME_CS: track 0.00 -> 15.6 mm, vias 0 -> 2
- net Net-(U1-EN): track 25.8 -> 39.6 mm, vias 0 -> 2
- net GND: track 17.9 -> 7.22 mm, vias 4 -> 23
- net /DIO1: track 35.4 -> 45.1 mm, vias 0 -> 2
- net Net-(U1-IO0): track 8.19 -> 17.4 mm, vias 0 -> 2
- net /RX1: track 0.00 -> 8.45 mm
- net /TX1: track 0.00 -> 8.08 mm
- net /BUSY: track 59.8 -> 64.3 mm, vias 0 -> 2
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Other:
- board size 30 x 65 mm -> 60 x 38 mm
- board text added: "COLD SWAP ONLY"
